File: ra-50.kicad_pcb (KiCad board)
At the start: 2 copper layers, 266.7 x 114.3 mm, 165 parts, among them J1 Conn_01x07, J2 Conn_01x07, SW1 MX-NoLED, SW10 MX-NoLED, SW11 MX-NoLED, SW12 MX-NoLED, SW13 MX-NoLED, SW14 MX-NoLED, SW14B1 Rotary_Encoder_Switch, SW15 MX-NoLED, SW16 MX-NoLED, SW17 MX-NoLED, SW18 MX-NoLED, SW19 MX-NoLED, SW2 MX-NoLED, SW20 MX-NoLED, SW21 MX-NoLED, SW22 MX-NoLED, SW23 MX-NoLED, SW24 MX-NoLED, SW25 MX-NoLED, SW26 MX-NoLED, SW27 MX-NoLED, SW28 MX-NoLED, SW29 MX-NoLED, SW3 MX-NoLED, SW30 MX-NoLED, SW31 MX-NoLED, SW32 MX-NoLED, SW33 MX-NoLED, SW34 MX-NoLED, SW35 MX-NoLED, SW36 MX-NoLED, SW37 MX-NoLED, SW38 MX-NoLED, SW39 MX-NoLED, SW4 MX-NoLED, SW40 MX-NoLED, SW41 MX-NoLED, SW42 MX-NoLED, SW43 MX-NoLED, SW44 MX-NoLED, SW45 MX-NoLED, SW46 MX-NoLED, SW47 MX-NoLED, SW48 MX-NoLED, SW49 MX-NoLED, SW5 MX-NoLED, SW50 MX-NoLED, SW51 MX-NoLED, SW52 MX-NoLED, SW53 MX-NoLED, SW54 MX-NoLED, SW55 MX-NoLED, SW56 MX-NoLED, SW57 MX-NoLED, SW58 MX-NoLED, SW59 MX-NoLED, SW6 MX-NoLED, SW60 MX-NoLED, SW61 MX-NoLED, SW62 MX-NoLED, SW63 MX-NoLED, SW64 MX-NoLED, SW65 MX-NoLED, SW66 MX-NoLED, SW67 MX-NoLED, SW68 MX-NoLED, SW69 MX-NoLED, SW7 MX-NoLED, SW8 MX-NoLED, SW9 MX-NoLED

Commit message: few routing done
Parts:
- moved D1 33.4 mm to (133.3, 75.4)
- moved D18 10.2 mm to (137.3, 68.3)
- moved D20 8.87 mm to (129.4, 66.7)
- moved D17 8.27 mm to (129.4, 74.7)
- moved D16 8.09 mm to (125.4, 73.8)
- moved D19 4.05 mm to (133.3, 67.5)
Routing:
- net Net-(D1-Pad2): track 12.2 -> 84.7 mm, vias 0 -> 1
- net Net-(D20-Pad2): track 151.1 -> 169.2 mm
- net Net-(D21-Pad2): track 169.9 -> 185.9 mm
- net Net-(D18-Pad2): track 124.5 -> 135.6 mm
- net Net-(D16-Pad2): track 89.9 -> 79.2 mm
- net Net-(D17-Pad2): track 113.9 -> 104.6 mm

Commit message: add more track route
Parts:
- moved J2 115.2 mm to (327.0, 107.7), turned to 180 degrees
- moved D5 65.5 mm to (141.3, 76.2)
- moved D4 58.4 mm to (137.3, 76.2)
- moved D7 48.4 mm to (149.2, 66.7)
- moved D6 43.9 mm to (145.3, 75.4)
- moved D3 40.7 mm to (141.3, 68.3)
- moved D2 33.5 mm to (145.3, 67.5)
Connections:
- net Net-(D27-Pad2) renamed D27
- D22 pad 2: Net-(D22-Pad2) -> D22
- D23 pad 2: Net-(D23-Pad2) -> D23
- D24 pad 2: Net-(D24-Pad2) -> D24
- D25 pad 2: Net-(D25-Pad2) -> D25
- D26 pad 2: Net-(D26-Pad2) -> D26
- D28 pad 2: Net-(D28-Pad2) -> D28
- J2 pad 2: Net-(J2-Pad2) -> D26
- J2 pad 3: Net-(J2-Pad3) -> D25
- J2 pad 4: Net-(J2-Pad4) -> D24
- J2 pad 5: Net-(J2-Pad5) -> D23
- J2 pad 6: Net-(J2-Pad6) -> D22
- J2 pad 7: Net-(J2-Pad7) -> D28
- SW22 pad 2: Net-(D22-Pad2) -> D22
- SW23 pad 2: Net-(D23-Pad2) -> D23
- SW24 pad 2: Net-(D24-Pad2) -> D24
- SW25 pad 2: Net-(D25-Pad2) -> D25
- SW26 pad 2: Net-(D26-Pad2) -> D26
- SW28 pad 2: Net-(D28-Pad2) -> D28
Routing:
- net D22: track 0.00 -> 265.1 mm
- net D23: track 0.00 -> 248.2 mm
- net D24: track 0.00 -> 231.3 mm
- net D25: track 0.00 -> 214.5 mm
- net D26: track 0.00 -> 197.6 mm
- net D28: track 0.00 -> 170.4 mm
- net D27: track 12.2 -> 160.8 mm
- net Net-(D7-Pad2): track 12.2 -> 87.2 mm
- net Net-(D65-Pad2): track 12.2 -> 76.5 mm
- net Net-(D66-Pad2): track 12.2 -> 57.8 mm
- net Net-(D6-Pad2): track 12.2 -> 57.7 mm
- net Net-(D2-Pad2): track 12.2 -> 55.2 mm
- net Net-(D5-Pad2): track 12.2 -> 41.0 mm
- net Net-(D67-Pad2): track 12.2 -> 39.1 mm
- net Net-(D3-Pad2): track 12.2 -> 35.5 mm
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
Commit message: add things, retrace, etc
Parts:
- added H1: MountingHole, locallib:2mm_hole, F.Cu at (83.8, 62.9)
- added H2: MountingHole, locallib:2mm_hole, F.Cu at (83.8, 76.9)
- added H3: MountingHole, locallib:2mm_hole, F.Cu at (212.7, 62.9)
- added H4: MountingHole, locallib:2mm_hole, F.Cu at (212.7, 76.9)
- added H5: MountingHole, locallib:2mm_hole, F.Cu at (341.1, 62.9)
- added H6: MountingHole, locallib:2mm_hole, F.Cu at (341.1, 76.9)
- added J3: Conn_01x05, Connector_PinHeader_1.00mm:PinHeader_1x05_P1.00mm_Vertical, F.Cu at (332.2, 155.2)
- added J4: Conn_01x12, Connector_PinHeader_1.00mm:PinHeader_1x12_P1.00mm_Vertical, F.Cu at (337.3, 64.3)
- added J5: Conn_01x20, Connector_PinHeader_1.00mm:PinHeader_1x20_P1.00mm_Vertical, F.Cu at (94.9, 78.6)
- J2: value Conn_01x07 -> Conn_01x05; footprint Connector_PinHeader_1.00mm:PinHeader_1x07_P1.00mm_Vertical -> Connector_PinHeader_1.00mm:PinHeader_1x05_P1.00mm_Vertical
- moved D1 37.5 mm to (128.0, 38.3)
- moved D15 37.5 mm to (112.1, 28.0)
- moved D18 37.5 mm to (132.0, 31.2)
- moved D19 37.5 mm to (128.0, 30.4)
- moved D2 37.5 mm to (139.9, 30.4)
- moved D3 37.5 mm to (136.0, 31.2)
- moved D32 37.5 mm to (116.1, 28.0)
- moved D33 37.5 mm to (116.1, 35.9)
- moved D34 37.5 mm to (112.1, 35.9)
- moved D4 37.5 mm to (132.0, 39.1)
- moved D43 37.5 mm to (92.3, 39.1)
- moved D44 37.5 mm to (88.3, 38.3)
- moved D45 37.5 mm to (96.3, 39.1)
- moved D46 37.5 mm to (100.2, 38.3)
- moved D47 37.5 mm to (92.3, 31.2)
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Connections:
- net D27 renamed /D27
- net Net-(D1-Pad2) renamed D1
- net Net-(D10-Pad2) renamed /D10
- net Net-(D11-Pad2) renamed /D11
- net Net-(D12-Pad2) renamed /D12
- net Net-(D13-Pad2) renamed /D13
- net Net-(D14-Pad2) renamed D14
- net Net-(D15-Pad2) renamed /D15
- net Net-(D16-Pad2) renamed /D16
- net Net-(D17-Pad2) renamed /D17
- net Net-(D18-Pad2) renamed /D18
- net Net-(D19-Pad2) renamed /D19
- net Net-(D2-Pad2) renamed /D2
- net Net-(D20-Pad2) renamed /D20
- net Net-(D21-Pad2) renamed /D21
- net Net-(D29-Pad2) renamed /D29
- net Net-(D3-Pad2) renamed /D3
- net Net-(D30-Pad2) renamed /D30
- net Net-(D31-Pad2) renamed /D31
- net Net-(D32-Pad2) renamed /D32
- net Net-(D33-Pad2) renamed /D33
- net Net-(D34-Pad2) renamed /D34
- net Net-(D35-Pad2) renamed /D35
- net Net-(D36-Pad2) renamed /D36
- net Net-(D37-Pad2) renamed /D37
- net Net-(D38-Pad2) renamed /D38
- net Net-(D39-Pad2) renamed /D39
- net Net-(D4-Pad2) renamed /D4
- net Net-(D40-Pad2) renamed /D40
- net Net-(D41-Pad2) renamed /D41
- net Net-(D42-Pad2) renamed D42
- net Net-(D43-Pad2) renamed D43
- net Net-(D44-Pad2) renamed D44
- net Net-(D45-Pad2) renamed D45
- net Net-(D46-Pad2) renamed D46
- net Net-(D47-Pad2) renamed D47
- net Net-(D48-Pad2) renamed D48
- net Net-(D49-Pad2) renamed D49
- net Net-(D5-Pad2) renamed /D5
- net Net-(D50-Pad2) renamed /D50
- net Net-(D51-Pad2) renamed /D51
- net Net-(D52-Pad2) renamed /D52
- net Net-(D53-Pad2) renamed /D53
- net Net-(D54-Pad2) renamed D54
- net Net-(D55-Pad2) renamed D55
- net Net-(D56-Pad2) renamed D56
- net Net-(D6-Pad2) renamed /D6
- net Net-(D64-Pad2) renamed D64
- net Net-(D65-Pad2) renamed D65
- net Net-(D66-Pad2) renamed D66
- net Net-(D67-Pad2) renamed D67
- net Net-(D68-Pad2) renamed D68
- net Net-(D69-Pad2) renamed D69
- net Net-(D7-Pad2) renamed /D7
- net Net-(D8-Pad2) renamed /D8
- net Net-(D9-Pad2) renamed /D9
- J2 pad 2: D26 -> D25
- J2 pad 3: D25 -> D24
- J2 pad 4: D24 -> D23
- J2 pad 5: D23 -> D22
Routing:
- net /D36: track 12.2 -> 328.3 mm
- net /D50: track 12.2 -> 328.1 mm
- net /D51: track 12.2 -> 310.2 mm
- net /D37: track 12.2 -> 307.7 mm
- net /D52: track 12.2 -> 292.3 mm
- net /D38: track 12.2 -> 287.2 mm
- net /D53: track 12.2 -> 274.4 mm
- net /D39: track 12.2 -> 266.7 mm
- net /D40: track 12.2 -> 246.1 mm
- net /D41: track 12.2 -> 225.0 mm
- net D64: track 43.4 -> 237.4 mm
- net D28: track 170.4 -> 41.9 mm
- net D26: track 197.6 -> 81.7 mm
- net D25: track 214.5 -> 102.8 mm
- net D54: track 12.2 -> 120.9 mm
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- removed copper zone on B.Cu, net GND
Other:
- outline, holes or cut-outs redrawn

Commit message: update
Parts:
- added J6: Conn_01x20, locallib:PinHeader_1x20_via, F.Cu at (105.4, 78.6)
- added J7: Conn_01x20, locallib:PinHeader_1x20_via, F.Cu at (125.5, 78.6)
- J5: footprint Connector_PinHeader_1.00mm:PinHeader_1x20_P1.00mm_Vertical -> locallib:PinHeader_1x20_via
- moved J5 9.52 mm to (85.4, 78.6)
Connections:
- net /D10 renamed D10
- net /D11 renamed D11
- net /D12 renamed D12
- net /D13 renamed D13
- net /D16 renamed D16
- net /D17 renamed D17
- net /D18 renamed D18
- net /D19 renamed D19
- net /D2 renamed D2
- net /D20 renamed D20
- net /D21 renamed D21
- net /D3 renamed D3
- net /D32 renamed D32
- net /D33 renamed D33
- net /D34 renamed D34
- net /D35 renamed D35
- net /D37 renamed D37
- net /D38 renamed D38
- net /D4 renamed D4
- net /D5 renamed D5
- net /D6 renamed D6
- net /D7 renamed D7
- net /D8 renamed D8
- net /D9 renamed D9
- D15 pad 2: /D15 -> D15
- D29 pad 2: /D29 -> D29
- D30 pad 2: /D30 -> D30
- D31 pad 2: /D31 -> D31
- J5 pad 17: Net-(J5-Pad17) -> D15
- J5 pad 18: Net-(J5-Pad18) -> D29
- J5 pad 19: Net-(J5-Pad19) -> D30
- J5 pad 20: Net-(J5-Pad20) -> D31
- SW15 pad 2: /D15 -> D15
- SW29 pad 2: /D29 -> D29
- SW30 pad 2: /D30 -> D30
- SW31 pad 2: /D31 -> D31
Routing:
- net /D39: track 266.7 -> 12.2 mm
- net /D40: track 246.1 -> 12.2 mm
- net /D53: track 274.4 -> 51.6 mm
- net /D52: track 292.3 -> 70.6 mm
- net /D51: track 310.2 -> 89.7 mm
- net /D50: track 328.1 -> 108.7 mm
- net /D36: track 328.3 -> 110.1 mm
- net /D41: track 225.0 -> 12.2 mm
- net D13: track 24.0 -> 207.8 mm
- net col12: track 139.4 -> 315.3 mm
- net D12: track 12.2 -> 178.9 mm
- net col11: track 215.1 -> 372.9 mm
- net D11: track 12.2 -> 161.9 mm
- net col10: track 290.2 -> 430.6 mm
- net D9: track 12.2 -> 149.4 mm
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Other:
- net class Default: trace_width 0.25 -> 0.2; via_dia 0.8 -> 0.6; via_drill 0.4 -> 0.3

Commit message: big revision
Parts:
- removed C1, C2, C3, C4, C5, C6, C7, C8: 0.1uF, Capacitor_SMD:C_0201_0603Metric_Pad0.64x0.40mm_HandSolder
- removed FlexCut1, FlexCut2: LongOvalCut, Keebio-Parts:LongOvalCut
- removed J1: Conn_01x07, Connector_PinHeader_1.00mm:PinHeader_1x07_P1.00mm_Vertical
- removed J2, J3: Conn_01x05, Connector_PinHeader_1.00mm:PinHeader_1x05_P1.00mm_Vertical
- removed J4: Conn_01x12, Connector_PinHeader_1.00mm:PinHeader_1x12_P1.00mm_Vertical
- removed J5, J6, J7: Conn_01x20, locallib:PinHeader_1x20_via
- removed UG-RGB1, UG-RGB2, UG-RGB3, UG-RGB4, UG-RGB5, UG-RGB6, UG-RGB7, UG-RGB8: WS2812B, LED_SMD:LED_WS2812B_PLCC4_5.0x5.0mm_P3.2mm
- added H10: flex_cut, locallib:LongOvalCut_225mmFlexCut, F.Cu at (212.7, 155.6)
- added H7: flex_cut, locallib:LongOvalCut_225mmFlexCut, F.Cu at (212.7, 98.4)
- added H8: flex_cut, locallib:LongOvalCut_225mmFlexCut, F.Cu at (212.7, 117.5)
- added H9: flex_cut, locallib:LongOvalCut_225mmFlexCut, F.Cu at (212.7, 136.5)
- added JST2: USB Conn, Connector_JST:JST_GH_SM04B-GHS-TB_1x04-1MP_P1.25mm_Horizontal, F.Cu at (315.6, 67.5)
- added RGB1: RGB Strip, Connector_PinSocket_2.54mm:PinSocket_1x03_P2.54mm_Vertical, B.Cu at (321.8, 64.9)
- D1, D10, D11, D12, D13, D14, D15, D16, D17, D18, D19, D2, D20, D21, D22, D23, D24, D25, D26, D27, D28, D29, D3, D30, D31, D32, D33, D34, D35, D36, D37, D38, D39, D4, D40, D41, D42, D43, D44, D45, D46, D47, D48, D49, D5, D50, D51, D52, D53, D54, D55, D56, D57, D58, D59, D6, D60, D61, D62, D63, D64, D65, D66, D67, D68, D69, D7, D8, D9: footprint Keebio-Parts:D_SOD123 -> master-Keebio-Parts:D_SOD123; moved to B.Cu
- H1, H2, H3, H4, H5, H6: value MountingHole -> 2mm
- JST1: footprint Connector_JST:JST_GH_SM04B-GHS-TB_1x04-1MP_P1.25mm_Horizontal -> Connector_PinHeader_2.54mm:PinHeader_1x04_P2.54mm_Vertical
- moved D68 224.3 mm to (325.4, 170.7)
- moved D28 223.9 mm to (328.6, 102.5), turned to 180 degrees
- moved D69 220.4 mm to (328.6, 170.7)
- moved D67 215.1 mm to (306.4, 170.7)
- moved D66 206.1 mm to (287.3, 170.7)
- moved D55 206.0 mm to (325.4, 140.6), turned to 180 degrees
- moved D13 201.9 mm to (325.4, 83.5), turned to 180 degrees
- moved D56 201.7 mm to (328.6, 140.6), turned to 180 degrees
- moved D14 201.1 mm to (328.6, 83.5), turned to 180 degrees
- moved D65 197.2 mm to (268.3, 170.7)
- moved D54 196.1 mm to (306.4, 140.6), turned to 180 degrees
- moved D12 186.9 mm to (306.4, 83.5), turned to 180 degrees
- moved D53 186.3 mm to (287.3, 140.6), turned to 180 degrees
- moved D62 186.1 mm to (209.6, 170.7)
- moved D64 185.6 mm to (249.2, 170.7)
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Connections:
- net D1 renamed /D1
- net D10 renamed /D10
- net D11 renamed /D11
- net D12 renamed /D12
- net D13 renamed /D13
- net D15 renamed /D15
- net D16 renamed /D16
- net D17 renamed /D17
- net D18 renamed /D18
- net D19 renamed /D19
- net D2 renamed /D2
- net D20 renamed /D20
- net D21 renamed /D21
- net D22 renamed /D22
- net D23 renamed /D23
- net D24 renamed /D24
- net D25 renamed /D25
- net D26 renamed /D26
- net D28 renamed /D28
- net D29 renamed /D29
- net D3 renamed /D3
- net D30 renamed /D30
- net D31 renamed /D31
- net D32 renamed /D32
- net D33 renamed /D33
- net D34 renamed /D34
- net D35 renamed /D35
- net D37 renamed /D37
- net D38 renamed /D38
- net D4 renamed /D4
- net D42 renamed /D42
- net D43 renamed /D43
- net D44 renamed /D44
- net D45 renamed /D45
- net D46 renamed /D46
- net D47 renamed /D47
- net D48 renamed /D48
- net D49 renamed /D49
- net D5 renamed /D5
- net D54 renamed /D54
- net D55 renamed /D55
- net D56 renamed /D56
- net D57 renamed /D57
- net D58 renamed /D58
- net D59 renamed /D59
- net D6 renamed /D6
- net D60 renamed /D60
- net D61 renamed /D61
- net D62 renamed /D62
- net D63 renamed /D63
- net D64 renamed /D64
- net D65 renamed /D65
- net D66 renamed /D66
- net D67 renamed /D67
- net D68 renamed /D68
- net D69 renamed /D69
- net D7 renamed /D7
- net D8 renamed /D8
- net D9 renamed /D9
- D14 pad 2: D14 -> /D14
- OL1 pad 1: SDA -> GND
- OL1 pad 2: SCL -> 5V
- OL1 pad 3: 5V -> SCL
- OL1 pad 4: GND -> SDA
- SW14 pad 2: D14 -> /D14
- SW14B1 pad S1: D14 -> col13
- SW14B1 pad S2: col13 -> /D14
- XA1 pad A5: Net-(XA1-PadA5) -> col11
- XA1 pad D0: Net-(XA1-PadD0) -> col9
- XA1 pad D1: Net-(XA1-PadD1) -> rgb
- XA1 pad D10: Net-(XA1-PadD10) -> col2
- XA1 pad D11: Net-(XA1-PadD11) -> col1
- XA1 pad D12: Net-(XA1-PadD12) -> col0
- XA1 pad D13: Net-(XA1-PadD13) -> col10
- XA1 pad D4: Net-(XA1-PadD4) -> col8
- XA1 pad D5: Net-(XA1-PadD5) -> col7
- XA1 pad D6: Net-(XA1-PadD6) -> col6
- XA1 pad D7: Net-(XA1-PadD7) -> col5
- XA1 pad D8: Net-(XA1-PadD8) -> col4
- XA1 pad D9: Net-(XA1-PadD9) -> col3
- XA1 pad MISO: Net-(XA1-PadMISO) -> col12
- XA1 pad MOSI: rotary_a -> rotary_b
- XA1 pad SCK: rotary_b -> col13
- XA1 pad SS: Net-(XA1-PadSS) -> rotary_a
Routing:
- net col7: track 607.1 -> 1034.8 mm
- net col6: track 544.1 -> 952.3 mm
- net col5: track 460.2 -> 828.3 mm
- net /D37: track 332.3 -> 15.9 mm
- net /D38: track 312.9 -> 15.9 mm
- net col3: track 172.2 -> 465.6 mm
- net col4: track 418.2 -> 709.0 mm
- net col8: track 614.8 -> 892.3 mm
- net col2: track 185.5 -> 431.6 mm
- net row4: track 0.00 -> 234.0 mm
- net row3: track 0.00 -> 231.8 mm
- net row2: track 0.00 -> 231.8 mm
- net row1: track 0.00 -> 231.8 mm
- net row0: track 0.00 -> 231.8 mm
- net col9: track 488.2 -> 695.3 mm
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Other:
- board size 266.7 x 114.3 mm -> 266.7 x 119.1 mm
- net class Default: clearance 0.2 -> 0.185
- rule trace_clearance: 0.2 -> 0.185
- board text added: "D+"
- board text added: "D-"
- board text added: "DO"
- board text added: "G"
- board text added: "V"

Commit message: final. or is it?
Parts:
- added JST3: HUB, Connector_PinHeader_2.54mm:PinHeader_1x04_P2.54mm_Vertical, F.Cu at (125.1, 66.0)
- added JST4: row hub, Connector_PinHeader_1.00mm:PinHeader_1x04_P1.00mm_Vertical, F.Cu at (292.6, 82.7)
- JST1: value USB Conn -> 2.54 THT
- JST2: value USB Conn -> JST 1.25
- RGB1: value RGB Strip -> RGB
- moved JST1 38.2 mm to (323.2, 66.0)
- moved SW14B1 21.6 mm to (336.3, 88.9), turned to 180 degrees
- moved RGB1 14.3 mm to (335.9, 67.3)
- moved XA1 14.3 mm to (311.7, 70.0)
- moved JST2 12.9 mm to (328.3, 69.8)
- moved R1 4.76 mm to (111.6, 72.1)
- moved R2 4.76 mm to (104.3, 72.1)
- moved USB1 4.76 mm to (108.0, 64.5)
- moved D14 2.55 mm to (330.6, 81.9), turned to 270 degrees
- moved H1 2.38 mm to (83.8, 62.9)
- moved H3 2.38 mm to (212.7, 62.9)
- moved H5 2.38 mm to (341.1, 62.9)
- moved H2 2.38 mm to (83.8, 76.9)
- moved H4 2.38 mm to (212.7, 76.9)
- moved H6 2.38 mm to (341.1, 76.9)
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Connections:
- SW14B1 pad S1: col13 -> /D14
- SW14B1 pad S2: /D14 -> col13
- XA1 pad A0: Net-(XA1-PadA0) -> row1
- XA1 pad A1: Net-(XA1-PadA1) -> row2
- XA1 pad A2: Net-(XA1-PadA2) -> row3
- XA1 pad A3: Net-(XA1-PadA3) -> row4
- XA1 pad A4: Net-(XA1-PadA4) -> row0
- XA1 pad MOSI: rotary_b -> rotary_a
- XA1 pad SS: rotary_a -> rotary_b
Routing:
- net GND: track 34.4 -> 283.4 mm
- net 5V: track 18.0 -> 251.1 mm
- net SDA: track 0.00 -> 230.5 mm
- net SCL: track 0.00 -> 228.7 mm
- net USB_GND: track 40.7 -> 247.1 mm
- net USB_DATA+: track 35.9 -> 235.6 mm
- net USB_DATA-: track 36.5 -> 230.2 mm
- net USB_VBUS: track 41.4 -> 234.7 mm, vias 0 -> 1
- net row4: track 234.0 -> 390.5 mm
- net row3: track 231.8 -> 348.8 mm
- net row2: track 231.8 -> 324.1 mm
- net row1: track 231.8 -> 300.1 mm
- net rotary_b: track 10.6 -> 31.5 mm
- net row0: track 231.8 -> 251.6 mm, vias 0 -> 1
- net rotary_a: track 18.7 -> 34.6 mm
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Other:
- board size 266.7 x 119.1 mm -> 266.7 x 123.8 mm
- net class Default: clearance 0.185 -> 0.2
- rule trace_clearance: 0.185 -> 0.2
- board text added: "b0"
- board text added: "b1"
- board text added: "b2"
- board text added: "b3"
- board text added: "b4"
- board text added: "b5"
- board text added: "b6"
- board text added: "b7"
- board text added: "c6"
- board text added: "c7"
- board text added: "d0"
- board text added: "d1"
- board text added: "d2"
- board text added: "d3"
- board text added: "d4"
- board text added: "d6"
- board text added: "d7"
- board text added: "e6"
- board text added: "f0"
- board text added: "f1"
- board text added: "f4"
- board text added: "f5"
- board text added: "f6"
- board text added: "f7"
