File: ra-50.sch (KiCad schematic (older format))
At the start: 163 parts, among them J1 Conn_01x07, J2 Conn_01x07, SW1 MX-NoLED, SW10 MX-NoLED, SW11 MX-NoLED, SW12 MX-NoLED, SW13 MX-NoLED, SW14 MX-NoLED, SW14B1 Rotary_Encoder_Switch, SW15 MX-NoLED, SW16 MX-NoLED, SW17 MX-NoLED, SW18 MX-NoLED, SW19 MX-NoLED, SW2 MX-NoLED, SW20 MX-NoLED, SW21 MX-NoLED, SW22 MX-NoLED, SW23 MX-NoLED, SW24 MX-NoLED, SW25 MX-NoLED, SW26 MX-NoLED, SW27 MX-NoLED, SW28 MX-NoLED, SW29 MX-NoLED, SW3 MX-NoLED, SW30 MX-NoLED, SW31 MX-NoLED, SW32 MX-NoLED, SW33 MX-NoLED, SW34 MX-NoLED, SW35 MX-NoLED, SW36 MX-NoLED, SW37 MX-NoLED, SW38 MX-NoLED, SW39 MX-NoLED, SW4 MX-NoLED, SW40 MX-NoLED, SW41 MX-NoLED, SW42 MX-NoLED, SW43 MX-NoLED, SW44 MX-NoLED, SW45 MX-NoLED, SW46 MX-NoLED, SW47 MX-NoLED, SW48 MX-NoLED, SW49 MX-NoLED, SW5 MX-NoLED, SW50 MX-NoLED, SW51 MX-NoLED, SW52 MX-NoLED, SW53 MX-NoLED, SW54 MX-NoLED, SW55 MX-NoLED, SW56 MX-NoLED, SW57 MX-NoLED, SW58 MX-NoLED, SW59 MX-NoLED, SW6 MX-NoLED, SW60 MX-NoLED, SW61 MX-NoLED, SW62 MX-NoLED, SW63 MX-NoLED, SW64 MX-NoLED, SW65 MX-NoLED, SW66 MX-NoLED, SW67 MX-NoLED, SW68 MX-NoLED, SW69 MX-NoLED, SW7 MX-NoLED, SW8 MX-NoLED, SW9 MX-NoLED

Commit message: add more track route
Connections:
- net D22: now reaches D22.2 (A), SW22.2 (ROW)
- net D22: now also J2.6 (Pin_6)
- net D23: now reaches D23.2 (A), SW23.2 (ROW)
- net D23: now also J2.5 (Pin_5)
- net D24: now reaches D24.2 (A), SW24.2 (ROW)
- net D24: now also J2.4 (Pin_4)
- net D25: now reaches D25.2 (A), SW25.2 (ROW)
- net D25: now also J2.3 (Pin_3)
- net D26: now reaches D26.2 (A), SW26.2 (ROW)
- net D26: now also J2.2 (Pin_2)
- net D27: now reaches D27.2 (A), SW27.2 (ROW)
- net D27: now also J2.1 (Pin_1)
- net D28: now reaches D28.2 (A), SW28.2 (ROW)
- net D28: now also J2.7 (Pin_7)
Changed lines of the file:
@@
 Text Label 850  4200 1    50   ~ 0
 D57
+Text Label 6050 1950 1    50   ~ 0
+D28
+Text Label 5650 1950 1    50   ~ 0
+D27
+Text Label 5250 1950 1    50   ~ 0
+D26
+Text Label 4850 1950 1    50   ~ 0
+D25
+Text Label 4450 1950 1    50   ~ 0
+D24
+Text Label 4050 1950 1    50   ~ 0
+D23
+Text Label 3650 1950 1    50   ~ 0
+D22
+Text GLabel 1350 6850 0    50   Input ~ 0
+D26
+Text GLabel 1350 6750 0    50   Input ~ 0
+D27
+Text GLabel 1350 7350 0    50   Input ~ 0
+D28
+Text GLabel 1350 6950 0    50   Input ~ 0
+D25
+Text GLabel 1350 7050 0    50   Input ~ 0
+D24
+Text GLabel 1350 7150 0    50   Input ~ 0
+D23
+Text GLabel 1350 7250 0    50   Input ~ 0
+D22
 $EndSCHEMATC

Commit message: add things, retrace, etc
Parts:
- added H1, H2, H3, H4, H5, H6: MountingHole, locallib:2mm_hole, symbol Mechanical:MountingHole
- added J3: Conn_01x05, Connector_PinHeader_1.00mm:PinHeader_1x05_P1.00mm_Vertical, symbol Connector_Generic:Conn_01x05
- added J4: Conn_01x12, Connector_PinHeader_1.00mm:PinHeader_1x12_P1.00mm_Vertical, symbol Connector_Generic:Conn_01x12
- added J5: Conn_01x20, Connector_PinHeader_1.00mm:PinHeader_1x20_P1.00mm_Vertical, symbol Connector_Generic:Conn_01x20
- J2: value Conn_01x07 -> Conn_01x05; footprint Connector_PinHeader_1.00mm:PinHeader_1x07_P1.00mm_Vertical -> Connector_PinHeader_1.00mm:PinHeader_1x05_P1.00mm_Vertical; symbol Connector_Generic:Conn_01x07 -> Connector_Generic:Conn_01x05
Connections:
- net D22: now also J2.5 (Pin_5); no longer J2.6 (Pin_6)
- net D23: now also J2.4 (Pin_4); no longer J2.5 (Pin_5)
- net D24: now also J2.3 (Pin_3); no longer J2.4 (Pin_4)
- net D25: now also J2.2 (Pin_2); no longer J2.3 (Pin_3)
- net D26: now also J2.1 (Pin_1); no longer J2.2 (Pin_2)
- net D27: no longer J2.1 (Pin_1)
- net D28: now also J4.11 (Pin_11); no longer J2.7 (Pin_7)
- net D57: now also J5.9 (Pin_9)
- net D58: now also J5.10 (Pin_10)
- net D59: now also J5.11 (Pin_11)
- net D60: now also J5.12 (Pin_12)
- net D61: now also J5.13 (Pin_13)
- net D62: now also J5.14 (Pin_14)
- net D63: now also J5.15 (Pin_15)
- net col0: now also J5.8 (Pin_8)
- net D1: now reaches D1.2 (A), SW1.2 (ROW)
- net D1: now also J5.16 (Pin_16)
- net D2: now reaches D2.2 (A), SW2.2 (ROW)
- net D3: now reaches D3.2 (A), SW3.2 (ROW)
- net D4: now reaches D4.2 (A), SW4.2 (ROW)
- net D5: now reaches D5.2 (A), SW5.2 (ROW)
- net D6: now reaches D6.2 (A), SW6.2 (ROW)
- net D7: now reaches D7.2 (A), SW7.2 (ROW)
- net D8: now reaches D8.2 (A), SW8.2 (ROW)
- net D9: now reaches D9.2 (A), SW9.2 (ROW)
- net D10: now reaches D10.2 (A), SW10.2 (ROW)
- net D11: now reaches D11.2 (A), SW11.2 (ROW)
- net D12: now reaches D12.2 (A), SW12.2 (ROW)
- net D13: now reaches D13.2 (A), SW13.2 (ROW)
- net D14: now reaches D14.2 (A), SW14.2 (ROW), SW14B1.S1
- net D14: now also J4.12 (Pin_12)
- net D15: now reaches D15.2 (A), SW15.2 (ROW)
- net D16: now reaches D16.2 (A), SW16.2 (ROW)
- net D17: now reaches D17.2 (A), SW17.2 (ROW)
- net D18: now reaches D18.2 (A), SW18.2 (ROW)
- net D19: now reaches D19.2 (A), SW19.2 (ROW)
- net D20: now reaches D20.2 (A), SW20.2 (ROW)
- net D21: now reaches D21.2 (A), SW21.2 (ROW)
- net D29: now reaches D29.2 (A), SW29.2 (ROW)
- net D30: now reaches D30.2 (A), SW30.2 (ROW)
- net D31: now reaches D31.2 (A), SW31.2 (ROW)
- net D32: now reaches D32.2 (A), SW32.2 (ROW)
- net D33: now reaches D33.2 (A), SW33.2 (ROW)
- net D34: now reaches D34.2 (A), SW34.2 (ROW)
- net D35: now reaches D35.2 (A), SW35.2 (ROW)
- net D36: now reaches D36.2 (A), SW36.2 (ROW)
- net D37: now reaches D37.2 (A), SW37.2 (ROW)
- net D38: now reaches D38.2 (A), SW38.2 (ROW)
- net D39: now reaches D39.2 (A), SW39.2 (ROW)
- net D40: now reaches D40.2 (A), SW40.2 (ROW)
- net D41: now reaches D41.2 (A), SW41.2 (ROW)
- net D42: now reaches D42.2 (A), SW42.2 (ROW)
- net D42: now also J4.10 (Pin_10)
- net D43: now reaches D43.2 (A), SW43.2 (ROW)
- net D43: now also J5.6 (Pin_6)
- net D44: now reaches D44.2 (A), SW44.2 (ROW)
- net D44: now also J5.7 (Pin_7)
- net D45: now reaches D45.2 (A), SW45.2 (ROW)
- net D45: now also J5.5 (Pin_5)
- net D46: now reaches D46.2 (A), SW46.2 (ROW)
- net D46: now also J5.4 (Pin_4)
- net D47: now reaches D47.2 (A), SW47.2 (ROW)
- net D47: now also J5.3 (Pin_3)
- net D48: now reaches D48.2 (A), SW48.2 (ROW)
- net D48: now also J5.2 (Pin_2)
- net D49: now reaches D49.2 (A), SW49.2 (ROW)
- net D49: now also J5.1 (Pin_1)
- net D50: now reaches D50.2 (A), SW50.2 (ROW)
- net D51: now reaches D51.2 (A), SW51.2 (ROW)
- net D52: now reaches D52.2 (A), SW52.2 (ROW)
- net D53: now reaches D53.2 (A), SW53.2 (ROW)
- net D54: now reaches D54.2 (A), SW54.2 (ROW)
- net D54: now also J4.9 (Pin_9)
- net D55: now reaches D55.2 (A), SW55.2 (ROW)
- net D55: now also J4.8 (Pin_8)
- net D56: now reaches D56.2 (A), SW56.2 (ROW)
- net D56: now also J4.7 (Pin_7)
- net D64: now reaches D64.2 (A), SW64.2 (ROW)
- net D64: now also J3.1 (Pin_1), J4.5 (Pin_5)
- net D65: now reaches D65.2 (A), SW65.2 (ROW)
- net D65: now also J3.2 (Pin_2), J4.4 (Pin_4)
- net D66: now reaches D66.2 (A), SW66.2 (ROW)
- net D66: now also J3.3 (Pin_3), J4.3 (Pin_3)
- net D67: now reaches D67.2 (A), SW67.2 (ROW)
- net D67: now also J3.4 (Pin_4), J4.2 (Pin_2)
- net D68: now reaches D68.2 (A), SW68.2 (ROW)
- net D68: now also J3.5 (Pin_5), J4.1 (Pin_1)
- net D69: now reaches D69.2 (A), SW69.2 (ROW)
- net D69: now also J4.6 (Pin_6)
Other:
- moved on the sheet: J1

Commit message: update
Parts:
- added J6, J7: Conn_01x20, locallib:PinHeader_1x20_via, symbol Connector_Generic:Conn_01x20
- J5: footprint Connector_PinHeader_1.00mm:PinHeader_1x20_P1.00mm_Vertical -> locallib:PinHeader_1x20_via
Connections:
- net D10: now also J7.8 (Pin_8)
- net D11: now also J7.10 (Pin_10)
- net D12: now also J7.12 (Pin_12)
- net D13: now also J7.14 (Pin_14)
- net D15: now also J5.17 (Pin_17)
- net D16: now also J6.11 (Pin_11)
- net D17: now also J6.9 (Pin_9)
- net D18: now also J6.8 (Pin_8)
- net D19: now also J6.7 (Pin_7)
- net D2: now also J6.12 (Pin_12)
- net D20: now also J6.6 (Pin_6)
- net D21: now also J6.5 (Pin_5)
- net D29: now also J5.18 (Pin_18)
- net D3: now also J6.14 (Pin_14)
- net D30: now also J5.19 (Pin_19)
- net D31: now also J5.20 (Pin_20)
- net D32: now also J6.1 (Pin_1)
- net D33: now also J6.2 (Pin_2)
- net D34: now also J6.3 (Pin_3)
- net D35: now also J6.4 (Pin_4)
- net D37: now also J7.16 (Pin_16)
- net D38: now also J7.15 (Pin_15)
- net D4: now also J7.6 (Pin_6)
- net D5: now also J7.4 (Pin_4)
- net D6: now also J7.2 (Pin_2)
- net D7: now also J6.20 (Pin_20)
- net D8: now also J6.18 (Pin_18)
- net D9: now also J6.16 (Pin_16)
- net col1: now also J6.10 (Pin_10)
- net col10: now also J7.9 (Pin_9)
- net col11: now also J7.11 (Pin_11)
- net col12: now also J7.13 (Pin_13)
- net col2: now also J6.13 (Pin_13)
- net col3: now also J6.15 (Pin_15)
- net col4: now also J6.17 (Pin_17)
- net col5: now also J6.19 (Pin_19)
- net col6: now also J7.1 (Pin_1)
- net col7: now also J7.3 (Pin_3)
- net col8: now also J7.5 (Pin_5)
- net col9: now also J7.7 (Pin_7)
Other:
- moved on the sheet: J5, XA1
Changed lines of the file:
@@
 L arduino:Arduino_Micro_Socket XA1
 U 1 1 60EDE630
-P 5150 6650
-F 0 "XA1" H 5150 7887 60  0000 C CNN
-F 1 "Arduino_Micro_Socket" H 5150 7781 60  0000 C CNN
-F 2 "Arduino:Arduino_Micro_Socket" H 6950 10400 60  0001 C CNN
-F 3 "https://store.arduino.cc/arduino-micro" H 6950 10400 60  0001 C CNN
-	1    5150 6650
-	1    0    0    -1
-$EndComp
-Text GLabel 3850 7450 0    50   Input ~ 0
+P 5300 6700
+F 0 "XA1" H 5300 7937 60  0000 C CNN
+F 1 "Arduino_Micro_Socket" H 5300 7831 60  0000 C CNN
+F 2 "Arduino:Arduino_Micro_Socket" H 7100 10450 60  0001 C CNN
+F 3 "https://store.arduino.cc/arduino-micro" H 7100 10450 60  0001 C CNN
+	1    5300 6700
+	1    0    0    -1
+$EndComp
+Text GLabel 4000 7500 0    50   Input ~ 0
 5V
-Text GLabel 3850 7250 0    50   Input ~ 0
+Text GLabel 4000 7300 0    50   Input ~ 0
 GND
-NoConn ~ 3850 7350
-NoConn ~ 3850 7550
-NoConn ~ 3850 6950
-NoConn ~ 6450 7350
-NoConn ~ 6450 7450
+NoConn ~ 4000 7400
+NoConn ~ 4000 7600
+NoConn ~ 4000 7000
+NoConn ~ 6600 7400
+NoConn ~ 6600 7500
 Text GLabel 7550 5950 0    50   Input ~ 0
 SDA
@@
 	-1   0    0    1
 $EndComp
-Text GLabel 3850 7150 0    50   Input ~ 0
+Text GLabel 4000 7200 0    50   Input ~ 0
 GND
 Text GLabel 7250 1200 2    50   Input ~ 0
 GND
-Text GLabel 3850 6150 0    50   Input ~ 0
+Text GLabel 4000 6200 0    50   Input ~ 0
 SCL
-Text GLabel 3850 6050 0    50   Input ~ 0
+Text GLabel 4000 6100 0    50   Input ~ 0
 SDA
-Text GLabel 6450 7050 2    50   Input ~ 0
+Text GLabel 6600 7100 2    50   Input ~ 0
 rotary_b
-Text GLabel 6450 6950 2    50   Input ~ 0
+Text GLabel 6600 7000 2    50   Input ~ 0
 rotary_a
 $Comp
@@
 L Connector_Generic:Conn_01x20 J5
 U 1 1 612D088F
-P 2750 5550
-F 0 "J5" H 2830 5542 50  0000 L CNN
-F 1 "Conn_01x20" H 2830 5451 50  0000 L CNN
-F 2 "Connector_PinHeader_1.00mm:PinHeader_1x20_P1.00mm_Vertical" H 2750 5550 50  0001 C CNN
-F 3 "~" H 2750 5550 50  0001 C CNN
-	1    2750 5550
+P 1850 5700
+F 0 "J5" H 1800 6800 50  0000 L CNN
+F 1 "Conn_01x20" H 1450 6700 50  0000 L CNN
+F 2 "locallib:PinHeader_1x20_via" H 1850 5700 50  0001 C CNN
+F 3 "~" H 1850 5700 50  0001 C CNN
+	1    1850 5700
 	1    0    0    -1
 $EndComp
@@
 Text Label 5650 2700 1    50   ~ 0
 D41
-Text GLabel 2550 4650 0    50   Input ~ 0
+Text GLabel 1650 4800 0    50   Input ~ 0
 D49
-Text GLabel 2550 4750 0    50   Input ~ 0
+Text GLabel 1650 4900 0    50   Input ~ 0
 D48
-Text GLabel 2550 4850 0    50   Input ~ 0
+Text GLabel 1650 5000 0    50   Input ~ 0
 D47
-Text GLabel 2550 4950 0    50   Input ~ 0
+Text GLabel 1650 5100 0    50   Input ~ 0
 D46
-Text GLabel 2550 5050 0    50   Input ~ 0
+Text GLabel 1650 5200 0    50   Input ~ 0
 D45
-Text GLabel 2550 5150 0    50   Input ~ 0
+Text GLabel 1650 5300 0    50   Input ~ 0
 D43
-Text GLabel 2550 5250 0    50   Input ~ 0
+Text GLabel 1650 5400 0    50   Input ~ 0
 D44
-Text GLabel 2550 6050 0    50   Input ~ 0
+Text GLabel 1650 6200 0    50   Input ~ 0
 D63
-Text GLabel 2550 5950 0    50   Input ~ 0
+Text GLabel 1650 6100 0    50   Input ~ 0
 D62
-Text GLabel 2550 5850 0    50   Input ~ 0
+Text GLabel 1650 6000 0    50   Input ~ 0
 D61
-Text GLabel 2550 5750 0    50   Input ~ 0
+Text GLabel 1650 5900 0    50   Input ~ 0
 D60
-Text GLabel 2550 5650 0    50   Input ~ 0
+Text GLabel 1650 5800 0    50   Input ~ 0
 D59
-Text GLabel 2550 5550 0    50   Input ~ 0
+Text GLabel 1650 5700 0    50   Input ~ 0
 D58
-Text GLabel 2550 5450 0    50   Input ~ 0
+Text GLabel 1650 5600 0    50   Input ~ 0
 D57
-Text GLabel 2550 5350 0    50   Input ~ 0
+Text GLabel 1650 5500 0    50   Input ~ 0
 col0
-Text GLabel 2550 6150 0    50   Input ~ 0
+Text GLabel 1650 6300 0    50   Input ~ 0
 D1
 $Comp
@@
 	1    0    0    -1
 $EndComp
+Text GLabel 1650 6400 0    50   Input ~ 0
+D15
+Text GLabel 1650 6500 0    50   Input ~ 0
+D29
+Text GLabel 1650 6600 0    50   Input ~ 0
+D30
+Text GLabel 2200 5700 0    50   Input ~ 0
+col1
+Text GLabel 1650 6700 0    50   Input ~ 0
+D31
+Text GLabel 2200 4800 0    50   Input ~ 0
+D32
+Text GLabel 2200 4900 0    50   Input ~ 0
+D33
+Text GLabel 2200 5000 0    50   Input ~ 0
+D34
+Text GLabel 2200 5100 0    50   Input ~ 0
+D35
+Text GLabel 2200 5200 0    50   Input ~ 0
+D21
+Text GLabel 2200 5300 0    50   Input ~ 0
+D20
+Text GLabel 2200 5400 0    50   Input ~ 0
+D19
+Text GLabel 2200 5500 0    50   Input ~ 0
+D18
+Text GLabel 2200 5600 0    50   Input ~ 0
+D17
+Text GLabel 2200 5800 0    50   Input ~ 0
+D16
+Text GLabel 2200 5900 0    50   Input ~ 0
+D2
+Text GLabel 2200 6000 0    50   Input ~ 0
+col2
+Text GLabel 2200 6100 0    50   Input ~ 0
+D3
+Text GLabel 2750 5700 0    50   Input ~ 0
+D11
+Text GLabel 2750 5900 0    50   Input ~ 0
+D12
+Text GLabel 2750 6100 0    50   Input ~ 0
+D13
+Text GLabel 2200 6200 0    50   Input ~ 0
+col3
+Text GLabel 2200 6400 0    50   Input ~ 0
+col4
+Text GLabel 2750 5500 0    50   Input ~ 0
+D10
+$Comp
+L Connector_Generic:Conn_01x20 J6
+U 1 1 60F7AB70
+P 2400 5700
+F 0 "J6" H 2350 6800 50  0000 L CNN
+F 1 "Conn_01x20" H 2000 6700 50  0000 L CNN
+F 2 "locallib:PinHeader_1x20_via" H 2400 5700 50  0001 C CNN
+F 3 "~" H 2400 5700 50  0001 C CNN
+	1    2400 5700
+	1    0    0    -1
+$EndComp
+Text GLabel 2200 6600 0    50   Input ~ 0
+col5
+Text GLabel 2750 4800 0    50   Input ~ 0
+col6
+Text GLabel 2750 5000 0    50   Input ~ 0
+col7
+Text GLabel 2750 5200 0    50   Input ~ 0
+col8
+Text GLabel 2750 5400 0    50   Input ~ 0
+col9
+Text GLabel 2750 5600 0    50   Input ~ 0
+col10
+Text GLabel 2750 5800 0    50   Input ~ 0
+col11
+Text GLabel 2750 6000 0    50   Input ~ 0
+col12
+Text GLabel 2750 6200 0    50   Input ~ 0
+D38
+Text GLabel 2200 6700 0    50   Input ~ 0
+D7
+Text GLabel 2200 6500 0    50   Input ~ 0
+D8
+Text GLabel 2750 4900 0    50   Input ~ 0
+D6
+Text GLabel 2750 5100 0    50   Input ~ 0
+D5
+Text GLabel 2750 5300 0    50   Input ~ 0
+D4
+Text GLabel 2200 6300 0    50   Input ~ 0
+D9
+$Comp
+L Connector_Generic:Conn_01x20 J7
+U 1 1 6115908E
+P 2950 5700
+F 0 "J7" H 2900 6800 50  0000 L CNN
+F 1 "Conn_01x20" H 2550 6700 50  0000 L CNN
+F 2 "locallib:PinHeader_1x20_via" H 2950 5700 50  0001 C CNN
+F 3 "~" H 2950 5700 50  0001 C CNN
+	1    2950 5700
+	1    0    0    -1
+$EndComp
+Text GLabel 2750 6300 0    50   Input ~ 0
+D37
 $EndSCHEMATC

Commit message: big revision
Parts:
- removed C1, C2, C3, C4, C5, C6, C7, C8: 0.1uF, Capacitor_SMD:C_0201_0603Metric_Pad0.64x0.40mm_HandSolder, symbol Device:C_Small
- removed J1: Conn_01x07, Connector_PinHeader_1.00mm:PinHeader_1x07_P1.00mm_Vertical, symbol Connector_Generic:Conn_01x07
- removed J2, J3: Conn_01x05, Connector_PinHeader_1.00mm:PinHeader_1x05_P1.00mm_Vertical, symbol Connector_Generic:Conn_01x05
- removed J4: Conn_01x12, Connector_PinHeader_1.00mm:PinHeader_1x12_P1.00mm_Vertical, symbol Connector_Generic:Conn_01x12
- removed J5, J6, J7: Conn_01x20, locallib:PinHeader_1x20_via, symbol Connector_Generic:Conn_01x20
- removed UG-RGB1, UG-RGB2, UG-RGB3, UG-RGB4, UG-RGB5, UG-RGB6, UG-RGB7, UG-RGB8: WS2812B, LED_SMD:LED_WS2812B_PLCC4_5.0x5.0mm_P3.2mm, symbol ws2812b:WS2812B
- added H10, H7, H8, H9: flex_cut, locallib:LongOvalCut_225mmFlexCut, symbol Mechanical:MountingHole
- added JST2: USB Conn, Connector_JST:JST_GH_SM04B-GHS-TB_1x04-1MP_P1.25mm_Horizontal, symbol Connector_Generic:Conn_01x04
- added RGB1: RGB Strip, Connector_PinSocket_2.54mm:PinSocket_1x03_P2.54mm_Vertical, symbol Connector_Generic:Conn_01x03
- D1, D10, D11, D12, D13, D14, D15, D16, D17, D18, D19, D2, D20, D21, D22, D23, D24, D25, D26, D27, D28, D29, D3, D30, D31, D32, D33, D34, D35, D36, D37, D38, D39, D4, D40, D41, D42, D43, D44, D45, D46, D47, D48, D49, D5, D50, D51, D52, D53, D54, D55, D56, D57, D58, D59, D6, D60, D61, D62, D63, D64, D65, D66, D67, D68, D69, D7, D8, D9: footprint Keebio-Parts:D_SOD123 -> master-Keebio-Parts:D_SOD123
- H1, H2, H3, H4, H5, H6: value MountingHole -> 2mm
- JST1: footprint Connector_JST:JST_GH_SM04B-GHS-TB_1x04-1MP_P1.25mm_Horizontal -> Connector_PinHeader_2.54mm:PinHeader_1x04_P2.54mm_Vertical
Connections:
- net 5V: now also OL1.2 (SCL), RGB1.3 (Pin_3); no longer OL1.3 (VCC)
- net D14: now also SW14B1.S2; no longer SW14B1.S1
- net GND: now also OL1.1 (SDA), RGB1.1 (Pin_1); no longer OL1.4 (GND)
- net SCL: now also OL1.3 (VCC); no longer OL1.2 (SCL)
- net SDA: now also OL1.4 (GND); no longer OL1.1 (SDA)
- net USB_DATA+: now also JST2.2 (Pin_2)
- net USB_DATA-: now also JST2.3 (Pin_3)
- net USB_GND: now also JST2.1 (Pin_1)
- net USB_VBUS: now also JST2.4 (Pin_4)
- net col0: now also XA1.D12
- net col1: now also XA1.D11
- net col10: now also XA1.D13
- net col11: now also XA1.A5
- net col12: now also XA1.MISO (SPI_MISO)
- net col13: now also SW14B1.S1, XA1.SCK (SPI_SCK); no longer SW14B1.S2
- net col2: now also XA1.D10
- net col3: now also XA1.D9
- net col4: now also XA1.D8
- net col5: now also XA1.D7 (D7_INT4)
- net col6: now also XA1.D6
- net col7: now also XA1.D5
- net col8: now also XA1.D4
- net col9: now also XA1.D0 (D0_RX0)
- net rotary_a: now also XA1.SS (SPI_CS); no longer XA1.MOSI (SPI_MOSI)
- net rotary_b: now also XA1.MOSI (SPI_MOSI); no longer XA1.SCK (SPI_SCK)
- net rgb: now reaches XA1.D1 (D1_TX0)
- net rgb: now also RGB1.2 (Pin_2)
Other:
- moved on the sheet: H1, H2, H3, H4, H5, H6, OL1, R1, R2, USB1

Commit message: final. or is it?
Parts:
- added JST3: HUB, Connector_PinHeader_2.54mm:PinHeader_1x04_P2.54mm_Vertical, symbol Connector_Generic:Conn_01x04
- added JST4: row hub, Connector_PinHeader_1.00mm:PinHeader_1x04_P1.00mm_Vertical, symbol Connector_Generic:Conn_01x04
- JST1: value USB Conn -> 2.54 THT
- JST2: value USB Conn -> JST 1.25
Connections:
- net D14: now also SW14B1.S1; no longer SW14B1.S2
- net USB_DATA+: now also JST3.2 (Pin_2)
- net USB_DATA-: now also JST3.3 (Pin_3)
- net USB_GND: now also JST3.1 (Pin_1)
- net USB_VBUS: now also JST3.4 (Pin_4)
- net col13: now also SW14B1.S2; no longer SW14B1.S1
- net rotary_a: now also XA1.MOSI (SPI_MOSI); no longer XA1.SS (SPI_CS)
- net rotary_b: now also XA1.SS (SPI_CS); no longer XA1.MOSI (SPI_MOSI)
- net row0: now also XA1.A4
- net row1: now also XA1.A0, JST4.4 (Pin_4)
- net row2: now also XA1.A1, JST4.3 (Pin_3)
- net row3: now also XA1.A2, JST4.2 (Pin_2)
- net row4: now also XA1.A3, JST4.1 (Pin_1)
Other:
- moved on the sheet: JST1, JST2
Changed lines of the file:
@@
 Text GLabel 6300 750  1    50   Input ~ 0
 col13
-Text GLabel 6650 1100 0    50   Input ~ 0
+Text GLabel 6650 1300 0    50   Input ~ 0
 col13
 Text GLabel 7250 1100 2    50   Input ~ 0
@@
 	-1   0    0    -1
 $EndComp
-Wire Wire Line
-	6100 1200 6650 1200
-Connection ~ 6100 1200
 $Comp
 L arduino:Arduino_Micro_Socket XA1
@@
 Text GLabel 4000 6100 0    50   Input ~ 0
 SDA
+Text GLabel 6600 7200 2    50   Input ~ 0
+rotary_b
 Text GLabel 6600 7000 2    50   Input ~ 0
-rotary_b
-Text GLabel 6600 7200 2    50   Input ~ 0
 rotary_a
 Text Label 3650 4200 1    50   ~ 0
@@
 	1    0    0    -1
 $EndComp
-Wire Wire Line
-	6650 1200 6650 1300
 Text GLabel 6600 6600 2    50   Input ~ 0
 col0
@@
 L Connector_Generic:Conn_01x04 JST2
 U 1 1 610653AD
-P 7800 5050
-F 0 "JST2" H 7718 4641 50  0000 C CNN
-F 1 "USB Conn" H 7718 4724 39  0000 C CNN
-F 2 "Connector_JST:JST_GH_SM04B-GHS-TB_1x04-1MP_P1.25mm_Horizontal" H 7800 5050 50  0001 C CNN
-F 3 "~" H 7800 5050 50  0001 C CNN
-	1    7800 5050
+P 6300 5100
+F 0 "JST2" H 6218 4691 50  0000 C CNN
+F 1 "JST 1.25" H 6218 4774 39  0000 C CNN
+F 2 "Connector_JST:JST_GH_SM04B-GHS-TB_1x04-1MP_P1.25mm_Horizontal" H 6300 5100 50  0001 C CNN
+F 3 "~" H 6300 5100 50  0001 C CNN
+	1    6300 5100
 	-1   0    0    1
 $EndComp
-Text GLabel 8000 5150 2    50   Input ~ 0
+Text GLabel 6500 5200 2    50   Input ~ 0
 USB_GND
-Text GLabel 8000 4850 2    50   Input ~ 0
+Text GLabel 6500 4900 2    50   Input ~ 0
 USB_VBUS
-Text GLabel 8000 4950 2    50   Input ~ 0
+Text GLabel 6500 5000 2    50   Input ~ 0
 USB_DATA-
-Text GLabel 8000 5050 2    50   Input ~ 0
+Text GLabel 6500 5100 2    50   Input ~ 0
 USB_DATA+
 $Comp
 L Connector_Generic:Conn_01x04 JST1
 U 1 1 61073EEA
-P 7050 5050
-F 0 "JST1" H 6968 4641 50  0000 C CNN
-F 1 "USB Conn" H 6968 4724 39  0000 C CNN
-F 2 "Connector_PinHeader_2.54mm:PinHeader_1x04_P2.54mm_Vertical" H 7050 5050 50  0001 C CNN
-F 3 "~" H 7050 5050 50  0001 C CNN
-	1    7050 5050
+P 5550 5100
+F 0 "JST1" H 5468 4691 50  0000 C CNN
+F 1 "2.54 THT" H 5468 4774 39  0000 C CNN
+F 2 "Connector_PinHeader_2.54mm:PinHeader_1x04_P2.54mm_Vertical" H 5550 5100 50  0001 C CNN
+F 3 "~" H 5550 5100 50  0001 C CNN
+	1    5550 5100
 	-1   0    0    1
 $EndComp
-Text GLabel 7250 5150 2    50   Input ~ 0
+Text GLabel 5750 5200 2    50   Input ~ 0
 USB_GND
-Text GLabel 7250 4850 2    50   Input ~ 0
+Text GLabel 5750 4900 2    50   Input ~ 0
 USB_VBUS
-Text GLabel 7250 4950 2    50   Input ~ 0
+Text GLabel 5750 5000 2    50   Input ~ 0
 USB_DATA-
-Text GLabel 7250 5050 2    50   Input ~ 0
+Text GLabel 5750 5100 2    50   Input ~ 0
 USB_DATA+
+Wire Wire Line
+	6100 1200 6650 1200
+Wire Wire Line
+	6650 1200 6650 1100
+Connection ~ 6100 1200
+$Comp
+L Connector_Generic:Conn_01x04 JST3
+U 1 1 610E9C2E
+P 7050 5100
+F 0 "JST3" H 6968 4691 50  0000 C CNN
+F 1 "HUB" H 6968 4774 39  0000 C CNN
+F 2 "Connector_PinHeader_2.54mm:PinHeader_1x04_P2.54mm_Vertical" H 7050 5100 50  0001 C CNN
+F 3 "~" H 7050 5100 50  0001 C CNN
+	1    7050 5100
+	-1   0    0    1
+$EndComp
+Text GLabel 7250 5200 2    50   Input ~ 0
+USB_GND
+Text GLabel 7250 4900 2    50   Input ~ 0
+USB_VBUS
+Text GLabel 7250 5000 2    50   Input ~ 0
+USB_DATA-
+Text GLabel 7250 5100 2    50   Input ~ 0
+USB_DATA+
+$Comp
+L Connector_Generic:Conn_01x04 JST4
+U 1 1 61204192
+P 7800 5100
+F 0 "JST4" H 7718 4691 50  0000 C CNN
+F 1 "row hub" H 7718 4774 39  0000 C CNN
+F 2 "Connector_PinHeader_1.00mm:PinHeader_1x04_P1.00mm_Vertical" H 7800 5100 50  0001 C CNN
+F 3 "~" H 7800 5100 50  0001 C CNN
+	1    7800 5100
+	-1   0    0    1
+$EndComp
+Text GLabel 8000 4900 2    50   Input ~ 0
+row1
+Text GLabel 8000 5000 2    50   Input ~ 0
+row2
+Text GLabel 8000 5100 2    50   Input ~ 0
+row3
+Text GLabel 8000 5200 2    50   Input ~ 0
+row4
+Text GLabel 4000 6900 0    50   Input ~ 0
+row1
+Text GLabel 4000 6800 0    50   Input ~ 0
+row2
+Text GLabel 4000 6700 0    50   Input ~ 0
+row3
+Text GLabel 4000 6600 0    50   Input ~ 0
+row4
+Text GLabel 4000 6500 0    50   Input ~ 0
+row0
 $EndSCHEMATC
